Commit message: add an examples of ANYmal trotting

File: examples/anymal/urdf/anymal.urdf (robot description, URDF)
Before this commit: robot anymal, 23 links, 22 joints
Links:
- link LF_ADAPTER: geometry collision cylinder length=0.32125 radius=0.015; visual mesh filename=package://anymal_b_simple_description/meshes/anymal_foot.dae scale=0.001 0.001 0.001
- link LF_FOOT: geometry collision sphere radius=0.031
- link LF_HIP: geometry collision cylinder length=0.03 radius=0.045; collision cylinder length=0.1 radius=0.08
- link LF_SHANK: geometry collision box size=0.08 0.07 0.13; visual mesh filename=package://anymal_b_simple_description/meshes/anymal_shank_l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 scale=0.001 0.001 0.001
- link LF_THIGH: geometry collision box size=0.08 0.04 0.25; collision cylinder length=0.12 radius=0.06
- link LH_ADAPTER: geometry collision cylinder length=0.32125 radius=0.015; visual mesh filename=package://anymal_b_simple_description/meshes/anymal_foot.dae scale=0.001 0.001 0.001
- link LH_FOOT: geometry collision sphere radius=0.031
- link LH_HIP: geometry collision cylinder length=0.03 radius=0.045; collision cylinder length=0.1 radius=0.08
- link LH_SHANK: geometry collision box size=0.08 0.07 0.13; visual mesh filename=package://anymal_b_simple_description/meshes/anymal_shank_r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 scale=0.001 0.001 0.001
- link LH_THIGH: geometry collision box size=0.08 0.04 0.25; collision cylinder length=0.12 radius=0.06
- link RF_ADAPTER: geometry collision cylinder length=0.32125 radius=0.015; visual mesh filename=package://anymal_b_simple_description/meshes/anymal_foot.dae scale=0.001 0.001 0.001
- link RF_FOOT: geometry collision sphere radius=0.031
- link RF_HIP: geometry collision cylinder length=0.03 radius=0.045; collision cylinder length=0.1 radius=0.08
- link RF_SHANK: geometry collision box size=0.08 0.07 0.13; visual mesh filename=package://anymal_b_simple_description/meshes/anymal_shank_r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 scale=0.001 0.001 0.001
- link RF_THIGH: geometry collision box size=0.08 0.04 0.25; collision cylinder length=0.12 radius=0.06
- link RH_ADAPTER: geometry collision cylinder length=0.32125 radius=0.015; visual mesh filename=package://anymal_b_simple_description/meshes/anymal_foot.dae scale=0.001 0.001 0.001
- link RH_FOOT: geometry collision sphere radius=0.031
- link RH_HIP: geometry collision cylinder length=0.03 radius=0.045; collision cylinder length=0.1 radius=0.08
- link RH_SHANK: geometry collision box size=0.08 0.07 0.13; visual mesh filename=package://anymal_b_simple_description/meshes/anymal_shank_l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 scale=0.001 0.001 0.001
- link RH_THIGH: geometry collision box size=0.08 0.04 0.25; collision cylinder length=0.12 radius=0.06
- link base: geometry collision box size=0.1 0.1 0.07; collision box size=0.1 0.1 0.07
