Commit message: modify examples and README

File: examples/iiwa14/iiwa_description/urdf/iiwa14.urdf (robot description, URDF)
Before this commit: robot iiwa14, 11 links, 10 joints
Links:
- link iiwa_link_0: geometry collision mesh filename=package://iiwa_description/meshes/iiwa14/collision/link_0.s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; visual mesh filename=package://iiwa_description/meshes/iiwa14/visual/link_0.stl
- link iiwa_link_1: geometry collision mesh filename=package://iiwa_description/meshes/iiwa14/collision/link_1.s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; visual mesh filename=package://iiwa_description/meshes/iiwa14/visual/link_1.stl
- link iiwa_link_2: geometry collision mesh filename=package://iiwa_description/meshes/iiwa14/collision/link_2.s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; visual mesh filename=package://iiwa_description/meshes/iiwa14/visual/link_2.stl
- link iiwa_link_3: geometry collision mesh filename=package://iiwa_description/meshes/iiwa14/collision/link_3.s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; visual mesh filename=package://iiwa_description/meshes/iiwa14/visual/link_3.stl
- link iiwa_link_4: geometry collision mesh filename=package://iiwa_description/meshes/iiwa14/collision/link_4.s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; visual mesh filename=package://iiwa_description/meshes/iiwa14/visual/link_4.stl
- link iiwa_link_5: geometry collision mesh filename=package://iiwa_description/meshes/iiwa14/collision/link_5.s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; visual mesh filename=package://iiwa_description/meshes/iiwa14/visual/link_5.stl
- link iiwa_link_6: geometry collision mesh filename=package://iiwa_description/meshes/iiwa14/collision/link_6.s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; visual mesh filename=package://iiwa_description/meshes/iiwa14/visual/link_6.stl
- link iiwa_link_7: geometry collision mesh filename=package://iiwa_description/meshes/iiwa14/collision/link_7.s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; visual mesh filename=package://iiwa_description/meshes/iiwa14/visual/link_7.stl
