Commit message: refactoring: cleanup code

File: examples/anymal/anymal_b_simple_description/urdf/anymal.urdf (robot description, URDF)
Before this commit: robot anymal, 24 links, 23 joints
Links:
- removed link world
Joints:
- removed joint floating

File: test/urdf/anymal/anymal.urdf (robot description, URDF)
Before this commit: robot anymal, 23 links, 22 joints
Links:
- removed link world
- added link imu_link, mass 0.05; collision box size=0.058 0.058 0.022; visual box size=0.058 0.058 0.022
- link LF_ADAPTER: geometry collision cylinder length=0.32125 radius=0.015; visual mesh filename=package://anymal_b_simple_description/meshes/foot/anymal_fo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 scale=1 1 1
- link LF_FOOT: mass None -> 0.001; geometry collision sphere radius=0.031
- link LF_HIP: geometry collision cylinder length=0.03 radius=0.045; collision cylinder length=0.1 radius=0.08
- link LF_SHANK: geometry collision box size=0.08 0.07 0.13; visual mesh filename=package://anymal_b_simple_description/meshes/shank/anymal_s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 scale=1 1 1
- link LF_THIGH: geometry collision box size=0.08 0.04 0.25; collision cylinder length=0.12 radius=0.06
- link LH_ADAPTER: geometry collision cylinder length=0.32125 radius=0.015; visual mesh filename=package://anymal_b_simple_description/meshes/foot/anymal_fo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 scale=1 1 1
- link LH_FOOT: mass None -> 0.001; geometry collision sphere radius=0.031
- link LH_HIP: geometry collision cylinder length=0.03 radius=0.045; collision cylinder length=0.1 radius=0.08
- link LH_SHANK: geometry collision box size=0.08 0.07 0.13; visual mesh filename=package://anymal_b_simple_description/meshes/shank/anymal_s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 scale=1 1 1
- link LH_THIGH: geometry collision box size=0.08 0.04 0.25; collision cylinder length=0.12 radius=0.06
- link RF_ADAPTER: geometry collision cylinder length=0.32125 radius=0.015; visual mesh filename=package://anymal_b_simple_description/meshes/foot/anymal_fo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 scale=1 1 1
- link RF_FOOT: mass None -> 0.001; geometry collision sphere radius=0.031
- link RF_HIP: geometry collision cylinder length=0.03 radius=0.045; collision cylinder length=0.1 radius=0.08
- link RF_SHANK: geometry collision box size=0.08 0.07 0.13; visual mesh filename=package://anymal_b_simple_description/meshes/shank/anymal_s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 scale=1 1 1
- link RF_THIGH: geometry collision box size=0.08 0.04 0.25; collision cylinder length=0.12 radius=0.06
- link RH_ADAPTER: geometry collision cylinder length=0.32125 radius=0.015; visual mesh filename=package://anymal_b_simple_description/meshes/foot/anymal_fo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 scale=1 1 1
- link RH_FOOT: mass None -> 0.001; geometry collision sphere radius=0.031
- link RH_HIP: geometry collision cylinder length=0.03 radius=0.045; collision cylinder length=0.1 radius=0.08
- link RH_SHANK: geometry collision box size=0.08 0.07 0.13; visual mesh filename=package://anymal_b_simple_description/meshes/shank/anymal_s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 scale=1 1 1
- link RH_THIGH: geometry collision box size=0.08 0.04 0.25; collision cylinder length=0.12 radius=0.06
- link base: mass None -> 1e-6; geometry collision box size=0.1 0.1 0.07; collision box size=0.1 0.1 0.07
Joints:
- removed joint floating
- added joint imu_joint: type fixed, parent base, child imu_link, origin xyz=0.038 0.06245 0.1837 rpy=0 3.14159265359 0
