Commit message: fix icub model

File: examples/icub/icub_description/urdf/icub.urdf (robot description, URDF)
Before this commit: robot iCub, 48 links, 47 joints
Links:
- removed link chest_depth_frame
- removed link chest_rgb_frame
- removed link l_foot_front
- removed link l_foot_rear
- removed link neck_3
- removed link r_foot_front
- removed link r_foot_rear
- added link chest_skin_frame, mass 0
- added link codyco_balancing_world, mass 0
- added link l_foot, mass 0.5935; collision mesh filename=package://icub_description/meshes/upmc/collision/icub_simpl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 scale=1 1 1; visual mesh filename=package://icub_description/meshes/upmc/visual/icub_l_foot.d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 scale=1 1 1
- added link l_foot_dh_frame, mass 0
- added link l_forearm_dh_frame, mass 0
- added link l_gripper, mass 0
- added link l_hand_dh_frame, mass 0
- added link l_upper_arm_dh_frame, mass 0
- added link r_foot, mass 0.5935; collision mesh filename=package://icub_description/meshes/upmc/collision/icub_simpl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 scale=1 1 1; visual mesh filename=package://icub_description/meshes/upmc/visual/icub_r_foot.d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 scale=1 1 1
- added link r_foot_dh_frame, mass 0
- added link r_forearm_dh_frame, mass 0
- added link r_gripper, mass 0
- added link r_hand_dh_frame, mass 0
- added link r_upper_arm_dh_frame, mass 0
- added link torso, mass 0
- link chest: mass 5.771074695 -> 4.81; geometry collision mesh filename=package://icub_description/meshes/upmc/collision/icub_simpl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 scale=1 1 1; visual mesh filename=package://icub_description/meshes/upmc/visual/icub_chest.dae scale=1 1 1
- link head: mass 1.831737118 -> 1.33687; geometry collision mesh filename=package://icub_description/meshes/upmc/collision/icub_simpl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 scale=1 1 1; visual mesh filename=package://icub_description/meshes/upmc/visual/icub_head.dae scale=1 1 1
- link imu_frame: mass None -> 0
- link l_ankle_1: mass 0.346176903 -> 0.746; geometry collision mesh filename=package://icub_description/meshes/upmc/collision/icub_simpl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 scale=1 1 1; visual mesh filename=package://icub_description/meshes/upmc/visual/icub_l_ankle_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 scale=1 1 1
- link l_ankle_2: mass 1.011533592 -> 0.2675; geometry 
- link l_elbow_1: mass 0.217768231 -> 0.074; geometry 
- link l_forearm: mass 0.858696525 -> 0.525; geometry collision mesh filename=package://icub_description/meshes/upmc/collision/icub_simpl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 scale=1 1 1; visual mesh filename=package://icub_description/meshes/upmc/visual/icub_l_forear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 scale=1 1 1
- link l_hand: mass 0.249250207 -> 0.213; geometry collision mesh filename=package://icub_description/meshes/upmc/collision/icub_simpl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 scale=1 1 1; visual mesh filename=package://icub_description/meshes/upmc/visual/icub_l_hand.d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 scale=1 1 1
- link l_hip_1: mass 2.108461113 -> 0.754; geometry collision mesh filename=package://icub_description/meshes/upmc/collision/icub_simpl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 scale=1 1 1; visual mesh filename=package://icub_description/meshes/upmc/visual/icub_l_hip_1.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 scale=1 1 1
- link l_hip_2: mass 1.781270621 -> 0.526; geometry collision mesh filename=package://icub_description/meshes/upmc/collision/icub_simpl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 scale=1 1 1; visual mesh filename=package://icub_description/meshes/upmc/visual/icub_l_hip_2.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 scale=1 1 1
- link l_hip_3: mass 2.169151426 -> 0; geometry 
- link l_lower_leg: mass 5.063049414 -> 1.264; geometry collision mesh filename=package://icub_description/meshes/upmc/collision/icub_simpl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 scale=1 1 1; visual mesh filename=package://icub_description/meshes/upmc/visual/icub_l_shank.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 scale=1 1 1
- link l_shoulder_1: mass 1.376687449 -> 0.189; geometry collision mesh filename=package://icub_description/meshes/upmc/collision/icub_simpl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 scale=1 1 1; visual mesh filename=package://icub_description/meshes/upmc/visual/icub_l_should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 scale=1 1 1
- link l_shoulder_2: mass 0.304658373 -> 0.179; geometry collision mesh filename=package://icub_description/meshes/upmc/collision/icub_simpl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 scale=1 1 1; visual mesh filename=package://icub_description/meshes/upmc/visual/icub_l_should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 scale=1 1 1
- link l_shoulder_3: mass 0.242239185 -> 0.156157; geometry 
- link l_sole: mass None -> 0
- link l_upper_arm: mass 2.07285 -> 0.727843; geometry collision mesh filename=package://icub_description/meshes/upmc/collision/icub_simpl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 scale=1 1 1; visual mesh filename=package://icub_description/meshes/upmc/visual/icub_l_arm.dae scale=1 1 1
- link l_upper_leg: mass 0.968264435 -> 2.175; geometry collision mesh filename=package://icub_description/meshes/upmc/collision/icub_simpl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 scale=1 1 1; visual mesh filename=package://icub_description/meshes/upmc/visual/icub_l_thigh.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 scale=1 1 1
- link l_wrist_1: mass 0.032535096 -> 0; geometry 
- link neck_1: mass 0.359964395 -> 0; geometry collision mesh filename=package://icub_description/meshes/upmc/collision/icub_simpl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 scale=1 1 1; visual mesh filename=package://icub_description/meshes/upmc/visual/icub_neck_1.d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 scale=1 1 1
- link neck_2: mass 0.118740971 -> 0; geometry collision mesh filename=package://icub_description/meshes/upmc/collision/icub_simpl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 scale=1 1 1; visual mesh filename=package://icub_description/meshes/upmc/visual/icub_neck_2.d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 scale=1 1 1
- link r_ankle_1: mass 0.346176903 -> 0.746; geometry collision mesh filename=package://icub_description/meshes/upmc/collision/icub_simpl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 scale=1 1 1; visual mesh filename=package://icub_description/meshes/upmc/visual/icub_r_ankle_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 scale=1 1 1
- link r_ankle_2: mass 1.00828013 -> 0.2675; geometry 
- link r_elbow_1: mass 0.217609341 -> 0.074; geometry 
- link r_forearm: mass 0.854281652 -> 0.525; geometry collision mesh filename=package://icub_description/meshes/upmc/collision/icub_simpl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 scale=1 1 1; visual mesh filename=package://icub_description/meshes/upmc/visual/icub_r_forear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 scale=1 1 1
- link r_hand: mass 0.2499009 -> 0.213; geometry collision mesh filename=package://icub_description/meshes/upmc/collision/icub_simpl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 scale=1 1 1; visual mesh filename=package://icub_description/meshes/upmc/visual/icub_r_hand.d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 scale=1 1 1
- link r_hip_1: mass 2.134290199 -> 0.754; geometry collision mesh filename=package://icub_description/meshes/upmc/collision/icub_simpl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 scale=1 1 1; visual mesh filename=package://icub_description/meshes/upmc/visual/icub_r_hip_1.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 scale=1 1 1
- link r_hip_2: mass 1.779000764 -> 0.526; geometry collision mesh filename=package://icub_description/meshes/upmc/collision/icub_simpl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 scale=1 1 1; visual mesh filename=package://icub_description/meshes/upmc/visual/icub_r_hip_2.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 scale=1 1 1
- link r_hip_3: mass 2.1678368 -> 0; geometry 
- link r_lower_leg: mass 5.074105512 -> 1.264; geometry collision mesh filename=package://icub_description/meshes/upmc/collision/icub_simpl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 scale=1 1 1; visual mesh filename=package://icub_description/meshes/upmc/visual/icub_r_shank.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 scale=1 1 1
- link r_shoulder_1: mass 1.380716446 -> 0.189; geometry collision mesh filename=package://icub_description/meshes/upmc/collision/icub_simpl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 scale=1 1 1; visual mesh filename=package://icub_description/meshes/upmc/visual/icub_r_should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 scale=1 1 1
- link r_shoulder_2: mass 0.304658373 -> 0.179; geometry collision mesh filename=package://icub_description/meshes/upmc/collision/icub_simpl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 scale=1 1 1; visual mesh filename=package://icub_description/meshes/upmc/visual/icub_r_should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 scale=1 1 1
- link r_shoulder_3: mass 0.24467077 -> 0.155; geometry 
- link r_sole: mass None -> 0
- link r_upper_arm: mass 1.960447492 -> 0.729; geometry collision mesh filename=package://icub_description/meshes/upmc/collision/icub_simpl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 scale=1 1 1; visual mesh filename=package://icub_description/meshes/upmc/visual/icub_r_arm.dae scale=1 1 1
- link r_upper_leg: mass 0.980691904 -> 2.175; geometry collision mesh filename=package://icub_description/meshes/upmc/collision/icub_simpl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 scale=1 1 1; visual mesh filename=package://icub_description/meshes/upmc/visual/icub_r_thigh.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 scale=1 1 1
- link r_wrist_1: mass 0.032535096 -> 0; geometry 
- link root_link: mass 2.52649319 -> 4.72; geometry collision mesh filename=package://icub_description/meshes/upmc/collision/icub_simpl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 scale=1 1 1; visual mesh filename=package://icub_description/meshes/upmc/visual/icub_root_lin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 scale=1 1 1
- link torso_1: mass 1.714262538 -> 0; geometry collision mesh filename=package://icub_description/meshes/upmc/collision/icub_simpl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 scale=1 1 1; visual mesh filename=package://icub_description/meshes/upmc/visual/icub_lap_belt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 scale=1 1 1
- link torso_2: mass 1.374672951 -> 0; geometry 
Joints:
- removed joint base_link_fixed_joint
- removed joint chest_depth_frame_fixed_joint
- removed joint chest_rgb_frame_fixed_joint
- removed joint l_foot_front_ft_sensor
- removed joint l_foot_rear_ft_sensor
- removed joint neck_fixed_joint
- removed joint r_foot_front_ft_sensor
- removed joint r_foot_rear_ft_sensor
- added joint base_fixed_joint: type fixed, parent base_link, child root_link, origin xyz=0 0 0 rpy=0 -0 0, axis 0 0 0
- added joint chest_skin_frame_fixed_joint: type fixed, parent chest, child chest_skin_frame, origin xyz=-0.0055 -0.032 3.36778e-19 rpy=1.5708 -1.22465e-16 -3.14159, axis 0 0 0
- added joint codyco_balancing_world_fixed_joint: type fixed, parent l_foot, child codyco_balancing_world, origin xyz=-0.0353 -7.60894e-35 -0.001 rpy=3.14159 -0 0, axis 0 0 0
- added joint l_foot_dh_frame_fixed_joint: type fixed, parent l_foot, child l_foot_dh_frame, origin xyz=-0.0353 0 -0.001 rpy=0 1.5708 -0, axis 0 0 0
- added joint l_foot_ft_sensor: type fixed, parent l_ankle_2, child l_foot, origin xyz=0.017 0 0.042 rpy=0 -0 0, axis 0 0 0
- added joint l_forearm_dh_frame_fixed_joint: type fixed, parent l_forearm, child l_forearm_dh_frame, origin xyz=0 0.1373 8.4072e-18 rpy=0 -0 0, axis 0 0 0
- added joint l_gripper_joint: type fixed, parent l_hand, child l_gripper, origin xyz=0.0625 0 -0.016 rpy=0 -0 0, axis 0 0 0
- added joint l_hand_dh_frame_fixed_joint: type fixed, parent l_hand, child l_hand_dh_frame, origin xyz=0.0625 0 -0.016 rpy=0 -0 0, axis 0 0 0
- added joint l_upper_arm_dh_frame_fixed_joint: type fixed, parent l_upper_arm, child l_upper_arm_dh_frame, origin xyz=0 0 0.08428 rpy=-1.5708 0 0, axis 0 0 0
- added joint r_foot_dh_frame_fixed_joint: type fixed, parent r_foot, child r_foot_dh_frame, origin xyz=-0.0353 0 -0.001 rpy=0 1.5708 -0, axis 0 0 0
- added joint r_foot_ft_sensor: type fixed, parent r_ankle_2, child r_foot, origin xyz=0.017 0 0.042 rpy=0 -0 0, axis 0 0 0
- added joint r_forearm_dh_frame_fixed_joint: type fixed, parent r_forearm, child r_forearm_dh_frame, origin xyz=0 -0.1373 -8.4072e-18 rpy=0 -0 0, axis 0 0 0
- added joint r_gripper_joint: type fixed, parent r_hand, child r_gripper, origin xyz=0.0625 0 0.016 rpy=0 -0 0, axis 0 0 0
- added joint r_hand_dh_frame_fixed_joint: type fixed, parent r_hand, child r_hand_dh_frame, origin xyz=0.0625 0 0.016 rpy=0 -0 0, axis 0 0 0
- added joint r_upper_arm_dh_frame_fixed_joint: type fixed, parent r_upper_arm, child r_upper_arm_dh_frame, origin xyz=0 0 0.08428 rpy=1.5708 -0 3.14159, axis 0 0 0
- added joint torso_joint: type fixed, parent chest, child torso, origin xyz=0.00231 0.1933 -1.18362e-17 rpy=0 -0 0, axis 0 0 0
- joint imu_frame_fixed_joint: axis (none) -> 0 0 0; origin xyz=0.0034999999997785457 0.0054999999863750895 0.1013340000004441 rpy=-3.141592653589793 0 -1.570796326794897 -> xyz=0.0185 -0.1108 0.0066 rpy=1.5708 -0 0
- joint l_ankle_pitch: axis 0.0 1.0 0.0 -> 0 -1 6.12323e-17; limit lower=-0.7853981633974483 upper=0.7853981633974483 effort=50000 velocity=120.0 -> lower=-0.733038 upper=0.366519 effort=24 velocity=100; origin xyz=0 -0.0005000000000000004 -0.255989 rpy=0 0 0 -> xyz=-0.213 0 0 rpy=-1.5708 0 0
- joint l_ankle_roll: axis 1.0 0.0 0.0 -> 1 0 0; limit lower=-0.4363323129985824 upper=0.4363323129985824 effort=50000 velocity=120.0 -> lower=-0.418879 upper=0.418879 effort=11 velocity=100; origin xyz=-0.052750000000000005 -0.018200000000000008 -0.03500000000000003 rpy=0 0 0 -> xyz=0 0 0 rpy=0 -1.5708 0
- joint l_arm_ft_sensor: axis (none) -> 0 0 0; child l_shoulder_3 -> l_upper_arm; origin xyz=-0.004350133156978329 3.632573233880443e-07 -0.05430003872406172 rpy=0 0 0 -> xyz=0.015 9.36797e-18 0.068 rpy=0 -0 0; parent l_shoulder_2 -> l_shoulder_3
- joint l_elbow: axis -8.811824154381087e-08 -1.0000002733514628 4.4047361189014644e-08 -> 0 1 6.12323e-17; limit lower=-0.05235987755982989 upper=1.3089969389957472 effort=50000 velocity=120.0 -> lower=0.0959931 upper=1.85005 effort=20 velocity=100; origin xyz=0.009999930234919404 -0.001499647423428896 -0.12370033753758375 rpy=0 0 0 -> xyz=0 0 0.08428 rpy=-6.12323e-17 0 0
- joint l_hip_pitch: axis 0.0 -1.0 0.0 -> 0 -1 6.12323e-17; limit lower=-0.7853981633974483 upper=2.007128639793479 effort=50000 velocity=120.0 -> lower=-0.767945 upper=2.30383 effort=84 velocity=100; origin xyz=0.0216 0.04045000000000001 0 rpy=0 0 0 -> xyz=0 -0.0681 -0.1199 rpy=0 1.5708 -3.14159
- joint l_hip_roll: axis 1.0 0.0 0.0 -> 1 0 -6.12323e-17; limit lower=-0.17453292519943295 upper=2.007128639793479 effort=50000 velocity=120.0 -> lower=-2.07694 upper=0.296706 effort=84 velocity=100; origin xyz=-0.04725 0.0331 -0.009000000000000008 rpy=0 0 0 -> xyz=0 0 0 rpy=0 -1.5708 3.14159
- joint l_hip_yaw: axis 0.0 0.0 1.0 -> 0 1 6.12323e-17; limit lower=-1.3962634015954636 upper=1.3962634015954636 effort=50000 velocity=120.0 -> lower=-1.37881 upper=1.37881 effort=40 velocity=100; origin xyz=0 -0.015000000000000006 -0.07090000000000007 rpy=0 0 0 -> xyz=0 0 -0.0665 rpy=-1.5708 -6.16298e-33 -6.12323e-17
- joint l_knee: axis 0.0 -1.0 0.0 -> 0 1.22465e-16 -1; limit lower=-1.2217304763960306 upper=0.08726646259971647 effort=50000 velocity=120.0 -> lower=-2.18166 upper=0.401426 effort=30 velocity=100; origin xyz=0.015 0.024900000000000012 -0.10619999999999996 rpy=0 0 0 -> xyz=0 -0.2236 -1.36916e-17 rpy=3.14159 -1.2326e-32 1.5708
- joint l_leg_ft_sensor: axis (none) -> 0 0 0; origin xyz=0.036699999999999997 0 -0.08969999999999995 rpy=0 0 0 -> xyz=0 0 0.0665 rpy=0 -0 0
- joint l_shoulder_pitch: axis 3.323079797673039e-07 0.9999999783534342 1.4452224303407313e-07 -> 0 -1 5.55112e-17; limit lower=-1.53588974175501 upper=0.22689280275926285 effort=50000 velocity=120.0 -> lower=-1.65806 upper=0.0872665 effort=84 velocity=100; origin xyz=-0.020835100000000002 0.0397423 0.1052029 rpy=0.25326162380993705 -1.1977334179319483e-07 -0.26179930184968747 -> xyz=0.00525 0.1433 -0.11026 rpy=1.309 5.55112e-17 1.5708
- joint l_shoulder_roll: axis 0.9999998262417684 2.0348252649342313e-07 -4.0230228454118944e-08 -> 0 1 6.12323e-17; limit lower=0.20943951023931956 upper=2.8448866807507573 effort=50000 velocity=120.0 -> lower=0 upper=2.80649 effort=84 velocity=100; origin xyz=0.004992849331690818 0.111499838456099 0.0002686502277366859 rpy=-0.17453296140985 -0.05374759931933852 0 -> xyz=0 0 0 rpy=1.5708 -1.11022e-16 -1.5708
- joint l_shoulder_yaw: axis 2.227647404040578e-08 -4.393786245948661e-08 -1.0000002566182309 -> 0 6.12323e-17 1; child l_upper_arm -> l_shoulder_3; limit lower=-0.8726646259971648 upper=1.3962634015954636 effort=50000 velocity=120.0 -> lower=-0.645772 upper=1.74533 effort=34 velocity=100; origin xyz=0 -4.2345248449371375e-07 -0.02249994137312443 rpy=0 0 0 -> xyz=4.33681e-19 1.73472e-18 0 rpy=6.12323e-17 -0 1.309; parent l_shoulder_3 -> l_shoulder_2
- joint l_sole_fixed_joint: axis (none) -> 0 0 0; origin xyz=0.05963 0 0 rpy=0 0 0 -> xyz=-0.0353 -7.60894e-35 -0.001 rpy=3.14159 -0 0; parent l_foot_rear -> l_foot
- joint l_wrist_pitch: axis -0.9999998262417684 -2.0348252649342313e-07 4.0230228454118944e-08 -> 0 1 6.12323e-17; limit lower=-1.2217304763960306 upper=0.4363323129985824 effort=50000 velocity=120.0 -> lower=-1.13446 upper=0.174533 effort=0.65 velocity=100; origin xyz=0.016600015934286182 0.002006895218072541 -0.10749964114254112 rpy=0 0 0 -> xyz=0 0.1373 8.4072e-18 rpy=1.5708 1.11022e-16 1.5708
- joint l_wrist_prosup: axis 2.227647404040578e-08 -4.393786245948661e-08 -1.0000002566182309 -> 0 1 6.12323e-17; limit lower=-1.53588974175501 upper=1.53588974175501 effort=50000 velocity=120.0 -> lower=-0.872665 upper=0.872665 effort=0.45 velocity=100; origin xyz=-0.014999870654177704 0.0019996435036348514 -0.055300063582479825 rpy=0 0 0 -> xyz=-0.015 0 0 rpy=1.5708 -1.11022e-16 -1.5708
- joint l_wrist_yaw: axis 8.811824154381087e-08 1.0000002733514628 -4.4047361189014644e-08 -> 0 0 1; limit lower=-0.2617993877991494 upper=0.6108652381980153 effort=50000 velocity=120.0 -> lower=-0.436332 upper=0.436332 effort=0.65 velocity=100; origin xyz=-0.016300121744729387 -0.0069993926815711816 0 rpy=0 0 0 -> xyz=0 0 0 rpy=0 -0 0
- joint neck_pitch: axis 0.0 -1.0 0.0 -> 0 1 6.12323e-17; child neck_2 -> neck_1; limit lower=-0.5235987755982988 upper=0.3839724354387525 effort=50000 velocity=120.0 -> lower=-0.698132 upper=0.523599 effort=20 velocity=100; origin xyz=0.00865 0 0.049000000000000016 rpy=0 0 0 -> xyz=0.00231 0.1933 -1.18362e-17 rpy=1.5708 1.11022e-16 1.5708; parent neck_1 -> chest
- joint neck_roll: axis 1.0 0.0 0.0 -> 0 -1 6.12323e-17; child neck_3 -> neck_2; limit lower=-0.3490658503988659 upper=0.3490658503988659 effort=50000 velocity=120.0 -> lower=-1.22173 upper=1.0472 effort=20 velocity=100; origin xyz=0 0 0.009500499999999995 rpy=0 0 0 -> xyz=0.0095 0 0 rpy=-1.5708 1.11022e-16 -1.5708; parent neck_2 -> neck_1
- joint neck_yaw: axis -1.6255499221370677e-21 -1.0999983743979075e-15 1.0 -> 0 -1 6.12323e-17; limit lower=-0.7853981633974483 upper=0.7853981633974483 effort=50000 velocity=120.0 -> lower=-0.959931 upper=0.959931 effort=20 velocity=100; origin xyz=0 0 0.06915000000000002 rpy=0 0 0 -> xyz=-5.77779e-34 0 0 rpy=-1.5708 -1.11022e-16 1.5708; parent neck_3 -> neck_2
- joint r_ankle_pitch: axis 0.0 1.0 0.0 -> 0 1 6.12323e-17; limit lower=-0.7853981633974483 upper=0.7853981633974483 effort=50000 velocity=120.0 -> lower=-0.733038 upper=0.366519 effort=24 velocity=100; origin xyz=0 0.0005000000000000004 -0.255989 rpy=0 0 0 -> xyz=-0.213 0 0 rpy=1.5708 -0 0
- joint r_ankle_roll: axis -1.0 0.0 0.0 -> -1 1.22465e-16 0; limit lower=-0.4363323129985824 upper=0.4363323129985824 effort=50000 velocity=120.0 -> lower=-0.418879 upper=0.418879 effort=11 velocity=100; origin xyz=-0.052750000000000005 0.018200000000000008 -0.03500000000000003 rpy=0 0 0 -> xyz=0 0 0 rpy=0 1.5708 3.14159
- joint r_arm_ft_sensor: axis (none) -> 0 0 0; child r_shoulder_3 -> r_upper_arm; origin xyz=-0.006849946385389875 2.1904996055921444e-07 -0.05429998157789099 rpy=0 0 0 -> xyz=0.015 -8.93429e-18 0.068 rpy=0 -0 0; parent r_shoulder_2 -> r_shoulder_3
- joint r_elbow: axis 2.4949582809984105e-07 -1.0000002733514362 2.7942487004772865e-08 -> 0 1 6.12323e-17; limit lower=-0.05235987755982989 upper=1.3089969389957472 effort=50000 velocity=120.0 -> lower=0.0959931 upper=1.85005 effort=20 velocity=100; origin xyz=0.009999931922603816 0.0014996401320274133 -0.1237003374895465 rpy=0 0 0 -> xyz=0 0 0.08428 rpy=3.14159 -0 3.14159
- joint r_hip_pitch: axis 0.0 -1.0 0.0 -> 0 1 6.12323e-17; limit lower=-0.7853981633974483 upper=2.007128639793479 effort=50000 velocity=120.0 -> lower=-0.767945 upper=2.30383 effort=84 velocity=100; origin xyz=0.0216 -0.040549999999999996 0 rpy=0 0 0 -> xyz=0 0.0681 -0.1199 rpy=0 1.5708 6.12323e-17
- joint r_hip_roll: axis -1.0 0.0 0.0 -> -1 0 6.12323e-17; limit lower=-0.17453292519943295 upper=2.007128639793479 effort=50000 velocity=120.0 -> lower=-2.07694 upper=0.296706 effort=84 velocity=100; origin xyz=-0.0473 -0.03310000000000001 -0.009000000000000008 rpy=0 0 0 -> xyz=0 0 0 rpy=0 1.5708 -6.12323e-17
- joint r_hip_yaw: axis 0.0 0.0 -1.0 -> 0 -1 6.12323e-17; limit lower=-1.3962634015954636 upper=1.3962634015954636 effort=50000 velocity=120.0 -> lower=-1.37881 upper=1.37881 effort=40 velocity=100; origin xyz=0 0.015000000000000006 -0.07090000000000007 rpy=0 0 0 -> xyz=0 0 -0.0665 rpy=-1.5708 -6.16298e-33 6.12323e-17
- joint r_knee: axis 0.0 -1.0 0.0 -> 0 1.22465e-16 -1; limit lower=-1.2217304763960306 upper=0.08726646259971647 effort=50000 velocity=120.0 -> lower=-2.18166 upper=0.401426 effort=30 velocity=100; origin xyz=0.015000000000000003 -0.0249 -0.10619999999999996 rpy=0 0 0 -> xyz=0 -0.2236 1.36916e-17 rpy=3.14159 -1.2326e-32 1.5708
- joint r_leg_ft_sensor: axis (none) -> 0 0 0; origin xyz=0.036699999999999997 0 -0.08969999999999995 rpy=0 0 0 -> xyz=0 0 0.0665 rpy=0 -0 0
- joint r_shoulder_pitch: axis 1.499044390054707e-07 0.9999999783534812 -1.2401537036188515e-07 -> 0 1 5.55112e-17; limit lower=-1.53588974175501 upper=0.22689280275926285 effort=50000 velocity=120.0 -> lower=-1.65806 upper=0.0872665 effort=84 velocity=100; origin xyz=-0.020835100000000002 -0.0397423 0.1052029 rpy=-0.25326164431680925 2.3014774394592079e-07 0.26179970938509745 -> xyz=0.00525 0.1433 0.11026 rpy=-1.309 -0 1.5708
- joint r_shoulder_roll: axis -0.9999998262417886 4.2105014356162707e-08 2.4630481189336084e-08 -> 0 -1 6.12323e-17; limit lower=0.20943951023931956 upper=2.8448866807507573 effort=50000 velocity=120.0 -> lower=0 upper=2.80649 effort=84 velocity=100; origin xyz=0.007489008185044645 -0.11150041046657978 0.0004027858966975245 rpy=0.17453306234069357 -0.053747792579130614 -6.132332688812785e-07 -> xyz=0 0 0 rpy=-1.5708 1.11022e-16 -1.5708
- joint r_shoulder_yaw: axis -3.787621790513063e-08 2.805197706068352e-08 1.0000002566182309 -> 0 6.12323e-17 -1; child r_upper_arm -> r_shoulder_3; limit lower=-0.8726646259971648 upper=1.3962634015954636 effort=50000 velocity=120.0 -> lower=-0.645772 upper=1.74533 effort=34 velocity=100; origin xyz=0 4.2183273077367467e-07 -0.022499941373153573 rpy=0 0 0 -> xyz=-4.33681e-19 0 0 rpy=3.14159 -0 1.309; parent r_shoulder_3 -> r_shoulder_2
- joint r_sole_fixed_joint: axis (none) -> 0 0 0; origin xyz=0.05963000000000001 0 0 rpy=0 0 0 -> xyz=-0.0353 -1.38778e-17 -0.001 rpy=3.14159 -0 0; parent r_foot_rear -> r_foot
- joint r_wrist_pitch: axis 0.9999998262417886 -4.2105014356162707e-08 -2.4630481189336084e-08 -> 0 1 6.12323e-17; limit lower=-1.2217304763960306 upper=0.4363323129985824 effort=50000 velocity=120.0 -> lower=-1.13446 upper=0.174533 effort=0.65 velocity=100; origin xyz=0.016299953353948633 -0.002007442890811839 -0.10750007971210637 rpy=0 0 0 -> xyz=0 -0.1373 -8.4072e-18 rpy=1.5708 1.11022e-16 1.5708
- joint r_wrist_prosup: axis -3.787621790513063e-08 2.805197706068352e-08 1.0000002566182309 -> 0 1 6.12323e-17; limit lower=-1.53588974175501 upper=1.53588974175501 effort=50000 velocity=120.0 -> lower=-0.872665 upper=0.872665 effort=0.45 velocity=100; origin xyz=-0.014999869468812953 -0.001999649905318951 -0.05530006367251966 rpy=0 0 0 -> xyz=0.015 0 0 rpy=1.5708 -1.11022e-16 -1.5708
- joint r_wrist_yaw: axis -2.4949582809984105e-07 1.0000002733514362 -2.7942487004772865e-08 -> 0 0 1; limit lower=-0.2617993877991494 upper=0.6108652381980153 effort=50000 velocity=120.0 -> lower=-0.436332 upper=0.436332 effort=0.65 velocity=100; origin xyz=-0.016300122874272734 0.0069993900510918194 0 rpy=0 0 0 -> xyz=0 0 0 rpy=0 -0 3.14159
- joint torso_pitch: axis 0.0 1.0 0.0 -> 0 1 6.12323e-17; child torso_2 -> torso_1; limit lower=-0.3141592653589793 upper=0.7853981633974483 effort=50000 velocity=120.0 -> lower=-0.383972 upper=1.46608 effort=36 velocity=100; origin xyz=0 0 0.07250000000000001 rpy=0 0 0 -> xyz=0 0 0 rpy=0 -1.5708 3.14159; parent torso_1 -> root_link
- joint torso_roll: axis -1.0 0.0 0.0 -> 0 1 6.12323e-17; child torso_1 -> torso_2; limit lower=-0.4014257279586958 upper=0.4014257279586958 effort=50000 velocity=120.0 -> lower=-0.680678 upper=0.680678 effort=80 velocity=100; origin xyz=0 0 0.0605 rpy=0 0 0 -> xyz=0.032 -2.67276e-51 0 rpy=1.5708 -1.11022e-16 -1.5708; parent root_link -> torso_1
- joint torso_yaw: axis 0.0 0.0 -1.0 -> 0 -1 6.12323e-17; limit lower=-0.7504915783575618 upper=0.7504915783575618 effort=50000 velocity=120.0 -> lower=-1.02974 upper=1.02974 effort=80 velocity=100; origin xyz=0 0 0.06447000000000001 rpy=0 0 0 -> xyz=-7.46298e-34 -0.0055 0 rpy=-1.5708 1.11022e-16 -1.5708
