Commit message: add test for surface contacts and fix icub model

File: examples/icub/icub_description/urdf/icub.urdf (robot description, URDF)
Before this commit: robot iCub, 56 links, 55 joints
Joints:
- joint neck_pitch: type revolute -> fixed
- joint neck_roll: type revolute -> fixed
- joint neck_yaw: type revolute -> fixed
