Commit message: add terrain examples and update README

File: bindings/python/robotoc_sim/rsc/terrain.urdf (robot description, URDF)
Before this commit: robot terrain, 1 links, 0 joints
Links:
- link terrainLink: geometry collision mesh filename=terrain.obj scale=0.25 0.25 0.5; visual mesh filename=terrain.obj scale=0.25 0.25 0.5
